File: ETAG_GEN3.brd (EAGLE design)
At the start: 68.6 x 53.3 mm, 94 parts, among them IC2 SAMD21G18A-AUT, J2 22-27-2021-02, J3 22-27-2021-02, Q1 FDN360P, Y1 32.768kHz, Y4 32,768Khz

Commit message: Updated files...
Parts:
- removed C12V: 1uF, rcl:C0805
- removed C19: 1uF, Condensatori:C0603-ROUND
- removed C1A, C1B: 4.7nF, rcl:C0603-ROUND
- removed C20, C21, C4: 100nF, Condensatori:C0603-ROUND
- removed C22_1, C22_2, C22_3, C22_4: 22uF, resistor:153CLV-0505
- removed C23, C24: 22p, Condensatori:C0603-ROUND
- removed C26: 10nF, Condensatori:C0603-ROUND
- removed C2A, C2B: 1.5nF, rcl:C0805
- removed C3A, C3B: 220nF, rcl:C0603-ROUND
- removed C3V: 4.7uF, rcl:C0805
- removed CAA, CAB, CNA, CNB: 1.2nF, rcl:C0805
- removed D1A, D1B, D2A, D2B, D3A, D3B, D4A, D4B, D5A, D5B: (no value), semicon-smd-ipc:SOT-23_2PAD
- removed D2: CD1206-S01575, Diodi:MINIMELF
- removed G1: 10MM_SM_COIN_CELL_CLIP, battery:10MM_SM_COIN_CELL_CLIP
- removed J2, J3: 22-27-2021-02, con-molex:6410-02
- removed LDO: MCP1703, microchip:SOT89
- removed R10, R12, R13, R9: 10k, Resistenze:R0603-ROUND
- removed R1A, R1B: 100K, rcl:C0603-ROUND
- removed R2A, R2B: 75K, rcl:C0603-ROUND
- removed R3A, R3B: 68K, rcl:C0603-ROUND
- removed R4A, R4B: 43K, rcl:C0603-ROUND
- removed R5A, R5B: 82, rcl:C0603-ROUND
- removed R6: 100R, Resistenze:R0603-ROUND
- removed R6A, R6B: 470K, rcl:C0603-ROUND
- removed R7: 360, rcl:C0603-ROUND
- removed RF_A, RF_B: U2270B, atmel:SO16
- removed U$4: SDMMC06132, microbuilder:06132
- removed U$6: LITE_TRAP_2POS, con-molex:LITE_TRAP_MINI
- removed Y1: 32.768kHz, microbuilder:CRYSTAL_8X3.8
- added BAT: 10MM_SM_COIN_CELL_CLIP, battery:10MM_SM_COIN_CELL_CLIP
- added C10, C9, CDIV1A, CDIV1B: 22pF, rcl:C0603-ROUND
- added C11, CAGNDA, CAGNDB: 1uF, rcl:C0603-ROUND
- added C2, C6, CBLKA, CBLKB, CDECA, CDECB, CXA, CXB: 100nF, rcl:C0603-ROUND
- added C3.3V, C5V: 10uF, rcl:C0805
- added C7, CDC2, CDCB, CFCAPA, CFCAPB: 10nF, rcl:C0603-ROUND
- added CDIV2A, CDIV2B: 1.5nF, rcl:C0603-ROUND
- added CE1, CE2, CE3: 150uF, rcl:E2-5
- added CON_P: LITE_TRAP_2POS, con-molex:LITE_TRAP_MINI
- added CREF: 4.7uF, Condensatori:SMC_A
- added CRES1A: 1.2nF, rcl:C0603-ROUND
- added CRES1B: 1nF, rcl:C0603-ROUND
- added CRES2A, CRES2B: 100pF, rcl:C0603-ROUND
- added CVA, CVB: 50pF, rcl:CTRIM3018_11
- added D1: CD1206-S01575, Diodi:MINIMELF
- added JPA, JPB, JP_PWR: NA, pinhead:1X02
- added L1: 2.2uH, rcl:SMT_COIL_INDUCTOR_4X4MM
- added R3: 10K, rcl:C0603-ROUND
- added R4, RP_INT, RP_SCL, RP_SDA: 10k, rcl:C0603-ROUND
- added RAA: 22, rcl:C0805
- added RAB: 22, rcl:R0805
- added RFA, RFB: EM4095, em-microelectronic:SO16
- added SD: SDMMC06132, microbuilder:06132
- added VREG: LM3671, Texas Instruments:SOT23-5L
- C1, C3, C8: device Condensatori:C0603-ROUND -> rcl:C0603-ROUND
- C5: value 4.7uF -> 100nF; device Condensatori:SMC_A -> rcl:C0603-ROUND
- ICSP6: value 3x2 M -> 3x2M
- L6, L7: device Protezione:0805 -> inductors:C0805K
- R1: value 10k -> 100; device Resistenze:R0603-ROUND -> rcl:C0603-ROUND
- R2, VDIV1, VDIV2: device Resistenze:R0603-ROUND -> rcl:C0603-ROUND
- RTC: value RTC_PCF8523T -> MC-RTC-RV-1805-C3-I2C; device microbuilder:SOIC8_150MIL -> Microcrystal-RTC:MC-RTC-C3
- Z5, Z6: value CG0603MLC-05E -> ESD_SUPRESSOR; device Protezione:CT/CN0603 -> diode:C0603-ROUND
- moved C5 27.2 mm to (43.1, 28.1), turned to 90 degrees
- moved RESET 10.3 mm to (32.1, 11.5), turned to 0 degrees
- moved R1 9.50 mm to (27.0, 17.6), turned to 0 degrees
- moved LED1 7.13 mm to (23.3, 17.6), turned to 270 degrees
- moved FD3 6.38 mm to (63.9, 45.2)
- moved C3 4.30 mm to (50.7, 43.0)
- moved FD1 3.62 mm to (2.10, 48.1)
- moved TP2 1.48 mm to (43.7, 25.2)
- moved TP1 1.48 mm to (45.9, 25.2)
- moved RTC 1.22 mm to (37.4, 44.6), turned to 90 degrees
- moved T_SD 0.84 mm to (35.4, 30.1), turned to 0 degrees
- moved Q1 0.81 mm to (11.8, 14.8)
- moved Z6 0.70 mm to (17.4, 25.7)
- moved L7 0.50 mm to (13.2, 27.6)
- moved R2 0.22 mm to (42.3, 20.0)
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- renumbered AD to HDR_AD, HEADER_IOH to HDR_IOH, HEADER_IOL to HDR_IOL, HEADER_POWER to HDR_POWER, IC2 to MCU, ICSP to ICSP6, ICSP! to ICSP10, U$9 to SW1
Connections:
- removed net +5V: HDR_POWER.5, ICSP6.2
- removed net HEADER_AD: HDR_AD.1
- removed net N$21: CNB.2, RF_B.4
- removed net N$23: D4B.P$1, R5B.1, RF_B.9
- removed net N$24: CAB.2, D1B.P$2, RF_B.8
- removed net N$25: CAB.1, D5B.P$2, J3.2, R1B.1, R2B.2
- removed net N$26: R4B.2, RF_B.15
- removed net N$27: C22_4.+, R3B.1, RF_B.14, RF_B.5, RF_B.6
- removed net N$28: D1B.P$1, D2B.P$1, R1B.2
- removed net N$29: D3B.P$2, D4B.P$2, R2B.1
- removed net N$30: C1B.2, D2B.P$2, D3B.P$1, R3B.2, R4B.1
- removed net N$40: CAA.2, D1A.P$2, RF_A.8
- removed net N$41: CAA.1, D5A.P$2, J2.1, R1A.1, R2A.2
- removed net N$43: R4A.2, RF_A.15
- removed net N$44: C22_3.+, R3A.1, RF_A.14, RF_A.5, RF_A.6
- removed net N$56: HDR_POWER.1
- new net CVB: CDIV1B.1, CRES1B.2, CRES2B.2, CVB.+, JPB.1
- new net N$16: CXB.1, RAB.2, RFB.3
- new net N$6: CDC2.1, RFA.16
- new net N$7: CRES1B.1, CRES2B.1, CVB.-, RFB.6
- new net N$8: CDIV1B.2, CDIV2B.1, RFB.8
- new net N$9: CDCB.1, RFB.16
- new net SW: L1.P$1, VREG.5
- net +3V3: now also C2.2, C3.3V.1, C5.1, D1.C, L1.P$2, R4.2, RP_INT.2, RP_SCL.2, RP_SDA.2, RTC.P$1, VREG.4; no longer C20.1, C3.2, C3V.1, D2.C, LDO.OUT, R1.2, R12.2, R13.2, R9.2, RTC.8
- net 12_IN: now also CON_P.P$3, CON_P.P$4, JP_PWR.2; no longer U$6.P$3, U$6.P$4
- net GND: now also BAT.-, C10.1, C11.2, C2.1, C3.2, C3.3V.2, C5.2, C5V.2, C6.2, C7.2, C9.1, CAGNDA.2, CAGNDB.2, CBLKA.2, CBLKB.2, CDC2.2, CDCB.2, CDIV2A.2, CDIV2B.2, CE1.-, CE2.-, CE3.-, CFCAPA.2, CFCAPB.2, CON_P.P$1, CON_P.P$2, CREF.-, JP_PWR.1, R3.2, RFA.1, RFA.12, RFA.5, RFB.1, RFB.12, RFB.5, RTC.P$6, RTC.P$8, RTC.P$9, SD.3, SD.6, SD.GP, SD.GP3, VREG.2, Z5.1, Z6.1; no longer C12V.2, C19.2, C1A.1, C1B.1, C20.2, C21.2, C22_1.-, C22_2.-, C22_3.-, C22_4.-, C23.1, C24.1, C26.2, C2A.1, C2B.1, C3.1, C3A.1, C3B.1, C3V.2, C4.2, C5.-, G1.-, LDO.GND, R10.1, R6A.1, R6B.1, RF_A.1, RF_A.3, RF_A.7, RF_B.1, RF_B.3, RF_B.7, RTC.4, U$4.3, U$4.6, U$4.GP, U$4.GP3, U$6.P$1, U$6.P$2, Z5.2, Z6.2
- net N$1: now also R1.1; no longer R6.1
- net N$10: now also C6.1; no longer C21.1
- net N$11: now also CDECB.2, RFB.9; no longer CNA.2, RF_A.4
- net N$12: now also CRES1A.1, CRES2A.1, CVA.-, RFA.6; no longer C2A.2, CNA.1, D5A.P$1, R6A.2
- net N$13: now also CDIV1A.2, CDIV2A.1, RFA.8; no longer C1A.2, D2A.P$2, D3A.P$1, R3A.2, R4A.1
- net N$14: now also CDIV1A.1, CRES1A.2, CRES2A.2, CVA.+, JPA.1; no longer J2.2, R5A.2
- net N$15: now also CDECB.1, RFB.10; no longer J3.1, R5B.2
- net N$18: now also CDECA.2, RFA.9; no longer D1A.P$1, D2A.P$1, R1A.2
- net N$19: now also CDECA.1, RFA.10; no longer C3B.2, RF_B.16
- net N$2: now also CFCAPB.1, RFB.15; no longer RTC.2, Y1.P$4
- net N$20: now also CXA.1, RAA.2, RFA.3; no longer D3A.P$2, D4A.P$2, R2A.1
- net N$22: now also JPB.2, RAB.1; no longer C2B.2, CNB.1, D5B.P$1, R6B.2
- net N$3: now also CAGNDB.1, RFB.11; no longer RTC.1, Y1.P$1
- net N$35: now also JPA.2, RAA.1; no longer D4A.P$1, R5A.1, RF_A.9
- net N$4: now also CFCAPA.1, RFA.15; no longer C22_1.+, R7.2, RF_A.12, RF_B.12
- net N$5: now also CAGNDA.1, RFA.11; no longer C3A.2, RF_A.16
- net PA00_XIN32: now also C9.2; no longer C23.2
- net PA01_XOUT32: now also C10.2; no longer C24.2
- net PA02_AIN0: now also HDR_AD.1
- net PA03_AREFA: now also C3.1, CREF.+; no longer C4.1, C5.+
- net PA21_INT&SDCS: now also RP_INT.1, RTC.P$3, SD.1; no longer R9.1, RTC.7, U$4.1
- net PA22_SDA: now also RP_SDA.1, RTC.P$5; no longer R13.1, RTC.5
- net PA23_SCL: now also RP_SCL.1, RTC.P$4; no longer R12.1, RTC.6
- net PA27_TX_LED: now also R1.2; no longer R6.2
- net PA28_2FETS: now also R3.1; no longer R10.2
- net PA6_RFID_SHD: now also RFA.14; no longer RF_A.13
- net PA7_RFID_SHD2: now also RFB.14; no longer RF_B.13
- net PB03_RFIDIN: now also RFA.13, RFB.13; no longer RF_A.2, RF_B.2
- net PB10_S4_SPI_MOSI: now also SD.2; no longer U$4.2
- net PB11_S4_SPI_SCK: now also SD.5; no longer U$4.5
- net PB12_S4_SPI_MISO: now also SD.7; no longer U$4.7
- net RESET: now also D1.A, R4.1; no longer D2.A, R1.1
- net TARGET_USB_N: now also Z6.2; no longer Z6.1
- net TARGET_USB_P: now also Z5.2; no longer Z5.1
- net VBAT1: now also BAT.+@1, BAT.+@2, RTC.P$7; no longer G1.+@1, G1.+@2, RTC.3
- net VDD: now also SD.4; no longer U$4.4
- net VDDCORE: now also C11.1; no longer C19.1
- net V_IN: now also C5V.1, CBLKA.1, CBLKB.1, CE1.+, CE2.+, CE3.+, CXA.2, CXB.2, HDR_POWER.5, ICSP6.2, RFA.4, RFA.7, RFB.4, RFB.7, VREG.1, VREG.3; no longer C12V.1, C22_2.+, LDO.IN, R7.1, RF_A.10, RF_A.11, RF_B.10, RF_B.11
- net XUSB: now also C7.1; no longer C26.1
Routing:
- net V_IN: track 125.8 -> 207.3 mm, vias 5 -> 4
- net +5V: track 51.0 -> 0.00 mm, vias 2 -> 0
- net N$41: track 26.1 -> 0.00 mm, vias 1 -> 0
- net N$25: track 23.5 -> 0.00 mm
- net CVB: track 0.00 -> 23.4 mm
- net N$4: track 25.1 -> 4.68 mm, vias 2 -> 0
- net N$27: track 19.4 -> 0.00 mm
- net PA03_AREFA: track 78.2 -> 58.8 mm, vias 1 -> 3
- net N$29: track 19.1 -> 0.00 mm, vias 3 -> 0
- net N$44: track 18.7 -> 0.00 mm
- net PA21_INT&SDCS: track 49.3 -> 31.4 mm, vias 1 -> 2
- net N$24: track 16.2 -> 0.00 mm, vias 2 -> 0
- net PA6_RFID_SHD: track 56.2 -> 71.5 mm, vias 2 -> 3
- net N$14: track 13.5 -> 28.7 mm, vias 1 -> 0
- net N$40: track 14.9 -> 0.00 mm, vias 2 -> 0
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Other:
- board text added: "+A"
- board text added: "-K"
- board text added: "1"
- board text added: "3.3V"
- board text added: "ANT 1"
- board text added: "ANT 2"
- board text added: "IOREF 3.3V"
- board text added: "L1 2.2uH"
- board text added: "Pin 1"
- board text added: "RFID Arduino University of Oklahoma March 2018"
- board text added: "V IN 5V"
- board text removed: "3V3"
- board text removed: "<- BATTERY +"
- board text removed: "IOREF"
- board text removed: "ON"
- board text removed: "Pin 1 ->"
- board text removed: "VIN"
