File: ETAG_GEN3.sch (EAGLE design)
At the start: 84 parts, among them CN2 PINHEAD-2x5-P1.27, IC2 SAMD21G18A-AUT, IC5 RTC_PCF8523T, IC6 EM4095, K1 G3VM-202J1, K2 G3VM-202J1, U1 SI1016CX-T1-GE3, U2 TC7SU04F, Y1 32.768kHz, Y4 32,768Khz

Commit message: Removed old design files
Parts:
- removed ANT1: ANT1_IN, con-molex:LITE_TRAP_2POS
- removed ANT2: ANT2_IN, con-molex:LITE_TRAP_2POS
- removed C2: 1u, Condensatori:0142_10NF_0603
- removed C6: 4.7u, Condensatori:0142_10NF_0603
- removed CAGND, CDC2, CDEC, CFCAP: (no value), rcl:C-US
- removed CDIV1, CDIV2, CRES: (no value), rcl:C-USC1206K
- removed C_BST: 0.1uF, rcl:C-US
- removed C_CO1, C_CO2: 22uF, rcl:C-EUC0805
- removed C_CO3: 10uF, rcl:C-EUC0805
- removed C_UP: 680pF, rcl:C-US
- removed C_VC1: 10uF, rcl:C-EUC1210
- removed D1: (no value), diode:ZENER-DIODESOD123
- removed IC5: RTC_PCF8523T, microbuilder:RTC_PCF8523T
- removed IC6: EM4095, em-microelectronic:EM4095
- removed JP1: (no value), pinhead:PINHD-1X2
- removed K1, K2: G3VM-202J1, relay:AQW21SOP
- removed L1: 22uH, rcl:L-EUSLF_10MM
- removed L2: 2.2uH, rcl:L-EU1008
- removed R-UP: 16K_1%, Resistenze:2022_CR0603FW104L
- removed R5, R8: 10k, Resistenze:0028_CR0603JW103L
- removed R_DN: 5.1K_0.1%, Resistenze:2339_
- removed SJ1, SJ2: (no value), jumper:SJW
- removed U$1: MCP1824T-3302E/OT, Microchip_By_element14_Batch_1:MCP1824T-3302E/OT
- removed U$3: BD93291EFJSOP8_W_GND, v-reg:BD93291EFJSOP8_W_GND
- removed U$5: USB-MINIB-5PIN, USB_miniB:USB-MINIB-5PIN
- removed U1: SI1016CX-T1-GE3, Vishay_By_element14_Batch_1:SI1016CX-T1-GE3
- removed U2: TC7SU04F, SparkFun-DigitalIC:INVERTER_SOT23-5
- removed VAR_C: TZB4Z100AB10R00, mylibrary:TZB4Z100AB10R00
- removed VDIV3: 200K, Resistenze:2022_CR0603FW104L
- removed VDIV_USB: ?, Resistenze:2339_
- added C12V: 1uF, rcl:C-USC0805
- added C1A, C1B: 4.7nF, rcl:C-US
- added C22_1, C22_2, C22_3, C22_4: 22uF, resistor:CPOL-US153CLV-0505
- added C2A, C2B: 1.5nF, rcl:C-USC0805
- added C3A, C3B: 220nF, rcl:C-US
- added C3V: 4.7uF, rcl:C-USC0805
- added CAA, CAB, CNA, CNB: 1.2nF, rcl:C-USC0805
- added D1A, D1B, D2A, D2B, D3A, D3B, D4A, D4B, D5A, D5B: (no value), semicon-smd-ipc:D-GLASS_MELF
- added J2, J3: 22-27-2021-02, con-molex:22-27-2021-02
- added LDO: MCP1703, microchip:MCP1703
- added MEM: AT45DB041BWIDE, SparkFun-DigitalIC:AT45DB041BWIDE
- added Q1: FDN360P, transistor-power:FDN360P
- added R1A, R1B: 100K, rcl:R-US_ROUND
- added R2A, R2B: 75K, rcl:R-US_ROUND
- added R3A, R3B: 68K, rcl:R-US_ROUND
- added R4A, R4B: 43K, rcl:R-US_ROUND
- added R5A, R5B: 82, rcl:R-US_ROUND
- added R6A, R6B: 470K, rcl:R-US_ROUND
- added RF_A, RF_B: U2270B, atmel:U2270B
- added RTC: RTC_PCF8523T, microbuilder:RTC_PCF8523T
- added TP1, TP2: TPTP15R, testpad:TPTP15R
- added USB: USB-MINIB-5PIN, USB_miniB:USB-MINIB-5PIN
- C26: value 10n -> 10nF
- C5: value 4u7 -> 4.7uF
- R2: value 330R -> 330
- R7: value (none) -> 360; device rcl:R-US_R1206 -> rcl:R-US_ROUND
- renumbered CN2 to ICSP!, IOH to HEADER_IOH, IOL to HEADER_IOL, POWER to HEADER_POWER
Connections:
- removed net +12V: C_VC1.2, HEADER_POWER.8, R5.1, U$3.P4_VIN, U$6G$2.S, U1.S2, VDIV3.2
- removed net +3.3_PSU: C_CO2.2, C_UP.1, L2.2, R-UP.2, U$9.S
- removed net +5_PSU: C_CO1.1, C_CO3.1, L1.1, U$3.P8_VO, U$9.S1
- removed net N$16: ANT2G$1.S, K2-1.D1
- removed net N$32: K1-1.A, K1-2.A, U2.Y
- removed net N$6: C_BST.1, U$3.P2_BST
- removed net N$7: C_UP.2, R-UP.1, R_DN.2, U$3.P6_FBL
- removed net N$8: R5.2, U$3.P3_EN
- removed net N$9: K1-2.D2, K2-1.D2, R7.1, SJ2.2
- removed net PA06_AIN6: HEADER_IOH.1, IC2.PA6/EIC/AIN6/SCOM0PAD2/TC1
- removed net PA7_RF_SWTICH: HEADER_IOH.2, IC2.PA7/EIC/AIN7/SCOM0PAD3/TC1, K2-1.A, K2-2.A, U2.A
- removed net X3.3V: C2.2, U$1.VOUT, U$9.O
- new net 12_IN: Q1.D, U$6G$2.S
- new net HEADER_AD: AD.1
- new net N$23: D4B.C, R5B.1, RF_B.COIL1
- new net N$24: CAB.2, D1B.A, RF_B.COIL2
- new net N$25: CAB.1, D5B.A, J3-2.S, R1B.1, R2B.2
- new net N$28: D1B.C, D2B.C, R1B.2
- new net N$29: D3B.A, D4B.A, R2B.1
- new net N$40: CAA.2, D1A.A, RF_A.COIL2
- new net N$41: CAA.1, D5A.A, J2-1.S, R1A.1, R2A.2
- new net N$43: R4A.2, RF_A.RF
- new net N$44: C22_3.+, R3A.1, RF_A.CFE, RF_A.MS, RF_A.VS
- new net PA7_RFID_SHD2: HEADER_IOH.2, IC2.PA7/EIC/AIN7/SCOM0PAD3/TC1, RF_B.STBY
- new net V_IN: C12V.1, C22_2.+, HEADER_POWER.8, LDO.VIN, R7.1, RF_A.DVS, RF_A.VEXT, RF_B.DVS, RF_B.VEXT, U$9.P, VDIV2.2
- net +3V3: now also C3V.1, LDO.VO, MEM.RST, MEM.VCC, RTC.VDD; no longer IC5.VDD, U$9.P, U2.VCC
- net +5V: no longer IC6.DVDD, IC6.VDD, U$9.P1
- net 2GND: now also USB.MTN1, USB.MTN2, USB.MTN3, USB.MTN4; no longer U$5.MTN1, U$5.MTN2, U$5.MTN3, U$5.MTN4
- net GND: now also C12V.2, C1A.1, C1B.1, C22_1.-, C22_2.-, C22_3.-, C22_4.-, C2A.1, C2B.1, C3A.1, C3B.1, C3V.2, LDO.GND, MEM.GND, MEM.WP, Q1.G, R6A.1, R6B.1, RF_A.DGND, RF_A.GND, RF_A.OE, RF_B.DGND, RF_B.GND, RF_B.OE, RTC.VSS, USB.GND; no longer C2.1, C6.1, CAGND.2, CDC2.2, CDIV2.2, CFCAP.2, C_CO1.2, C_CO2.1, C_CO3.2, C_VC1.1, D1.A, IC5.VSS, IC6.DVSS, IC6.MOD, IC6.VSS, R8.1, R_DN.1, U$1.GND, U$3.GNDPAD, U$3.P5_GND, U$5.GND, U1.S1, U2.GND
- net N$11: now also CNA.2, RF_A.INPUT; no longer CDIV1.1, CRES.2, K1-1.D2, K2-2.D2, SJ1.2, VAR_C.P$2
- net N$12: now also C2A.2, CNA.1, D5A.C, R6A.2; no longer CRES.1, IC6.ANT2, VAR_C.P$1
- net N$13: now also C1A.2, D2A.A, D3A.C, R3A.2, R4A.1; no longer CDIV1.2, CDIV2.1, IC6.DMOD_IN
- net N$14: now also J2-2.S, R5A.2; no longer ANT1G$1.S, K1-1.D1, SJ1.1
- net N$15: now also J3-1.S, R5B.2; no longer U1.D1, U1.G2, VDIV3.1
- net N$17: now also Q1.S, U$9.O; no longer CDC2.1, IC6.DC2
- net N$18: now also D1A.C, D2A.C, R1A.2; no longer CDEC.2, IC6.CDEC_OUT
- net N$19: now also C3B.2, RF_B.HIPASS; no longer CDEC.1, IC6.CDEC_IN
- net N$2: now also RTC.XO; no longer IC5.XO
- net N$20: now also D3A.A, D4A.A, R2A.1; no longer IC6.ANT1, R7.2
- net N$21: now also CNB.2, RF_B.INPUT; no longer D1.C, U1.D2, VDIV2.2
- net N$22: now also C2B.2, CNB.1, D5B.C, R6B.2; no longer K1-1.K, K1-2.K, K2-1.K, K2-2.K, R8.2
- net N$26: now also R4B.2, RF_B.RF; no longer L2.1, U$3.P7_SWL
- net N$27: now also C22_4.+, R3B.1, RF_B.CFE, RF_B.MS, RF_B.VS; no longer C_BST.2, L1.2, U$3.P1_SW
- net N$3: now also RTC.XI; no longer IC5.XI
- net N$30: now also C1B.2, D2B.A, D3B.C, R3B.2, R4B.1; no longer ANT2G$2.S, K2-2.D1
- net N$35: now also D4A.C, R5A.1, RF_A.COIL1; no longer ANT1G$2.S, K1-2.D1, SJ2.1
- net N$4: now also C22_1.+, R7.2, RF_A.VBATT, RF_B.VBATT; no longer CFCAP.1, IC6.FCAP
- net N$5: now also C3A.2, RF_A.HIPASS; no longer CAGND.1, IC6.AGND
- net PA02_AIN0: no longer AD.1, VDIV_USB.1
- net PA08_TCC0-W0_PA8: now also MEM.CS
- net PA21_INT&SDCS: now also RTC.!INT1/CLK; no longer IC5.!INT1/CLK
- net PA22_SDA: now also RTC.SDA; no longer IC5.SDA
- net PA23_SCL: now also RTC.SCL; no longer IC5.SCL
- net PA28_2FETS: no longer U1.G1
- net PA6_RFID_SHD: now also HEADER_IOH.1, IC2.PA6/EIC/AIN6/SCOM0PAD2/TC1, RF_A.STBY; no longer IC6.SHD
- net PB03_RFIDIN: now also RF_A.OUTPUT, RF_B.OUTPUT; no longer IC6.DMOD_OUT
- net PB10_S4_SPI_MOSI: now also MEM.SI
- net PB11_S4_SPI_SCK: now also MEM.SCK
- net PB12_S4_SPI_MISO: now also MEM.SO
- net PB22_DEBUG_TX: now also TP2.TP; no longer JP1.2
- net PB23_DEBUG_RX: now also TP1.TP; no longer JP1.1
- net TARGET_USB_N: now also USB.D-; no longer U$5.D-
- net TARGET_USB_P: now also USB.D+; no longer U$5.D+
- net VBAT1: now also RTC.VBAT; no longer IC5.VBAT
- net XUSB: now also U$9.S, USB.VBUS; no longer C6.2, U$1.VIN, U$1.~SHDN, U$5.VBUS, U$9.O1, VDIV_USB.2
Other:
- note added: "10"
- note added: "11"
- note added: "12"
- note added: "13"
- note added: "14"
- note added: "15"
- note added: "16"
- note added: "2"
- note added: "3"
- note added: "4"
- note added: "5"
- note added: "6"
- note added: "8"
- note added: "9"
- note added: "BAT"
- note added: "CFE"
- note added: "DGND"
- note added: "DVS"
- note added: "GND"
- note added: "HIPASS"
- note added: "INPUT"
- note added: "MS"
- note added: "OE"
- note added: "OUTPUT"
- note added: "RF"
- note added: "STBY"
- note added: "VEXT"
- note added: "VS"

Commit message: Updated files...
Parts:
- removed C12V: 1uF, rcl:C-USC0805
- removed C19: 1uF, Condensatori:0006_1UF_0603/GRM188R61E105KA12D
- removed C1A, C1B: 4.7nF, rcl:C-US
- removed C20, C21, C4: 100nF, Condensatori:0015_100NF_0603
- removed C22_1, C22_2, C22_3, C22_4: 22uF, resistor:CPOL-US153CLV-0505
- removed C23, C24: 22p, Condensatori:0014_22PF_0603
- removed C26: 10nF, Condensatori:0142_10NF_0603
- removed C2A, C2B: 1.5nF, rcl:C-USC0805
- removed C3A, C3B: 220nF, rcl:C-US
- removed C3V: 4.7uF, rcl:C-USC0805
- removed CAA, CAB, CNA, CNB: 1.2nF, rcl:C-USC0805
- removed D1A, D1B, D2A, D2B, D3A, D3B, D4A, D4B, D5A, D5B: (no value), semicon-smd-ipc:D-GLASS_MELF
- removed G1: 10MM_SM_COIN_CELL_CLIP, battery:10MM_SM_COIN_CELL_CLIP
- removed ICSP!: PINHEAD-2x5-P1.27, Connettori:0171_PH127-205DF055G00AROUND-PADS
- removed J2, J3: 22-27-2021-02, con-molex:22-27-2021-02
- removed LDO: MCP1703, microchip:MCP1703
- removed R10, R12, R13, R9: 10k, Resistenze:0028_CR0603JW103L
- removed R1A, R1B: 100K, rcl:R-US_ROUND
- removed R2A, R2B: 75K, rcl:R-US_ROUND
- removed R3A, R3B: 68K, rcl:R-US_ROUND
- removed R4A, R4B: 43K, rcl:R-US_ROUND
- removed R5A, R5B: 82, rcl:R-US_ROUND
- removed R6: 100R, Resistenze:0233_0R_0603
- removed R6A, R6B: 470K, rcl:R-US_ROUND
- removed R7: 360, rcl:R-US_ROUND
- removed RF_A, RF_B: U2270B, atmel:U2270B
- removed U$6: LITE_TRAP_2POS, con-molex:LITE_TRAP_2POS
- removed U$9: MFS201N-9-Z, switch:MFS201N-9-Z
- removed Y1: 32.768kHz, microbuilder:CRYSTAL8.0X3.8
- added BAT: 10MM_SM_COIN_CELL_CLIP, battery:10MM_SM_COIN_CELL_CLIP
- added C10, C9: 22pF, rcl:C-USROUND
- added C11: 1uF, rcl:C-USROUND
- added C2, C6: 100nF, rcl:C-USROUND
- added C3.3V, C5V: 10uF, rcl:C-USC0805
- added C7, CDCB, CFCAPA: 10nF, rcl:C-USROUND
- added CAGNDA, CAGNDB: 1uF, rcl:C-US
- added CBLKA, CBLKB, CDECA, CDECB, CXA, CXB: 100nF, rcl:C-US
- added CDC2, CFCAPB: 10nF, rcl:C-US
- added CDIV1A, CDIV1B: 22pF, rcl:C-US
- added CDIV2A: 1.5nF, rcl:C-USROUND
- added CDIV2B: 1.5nF, rcl:C-US
- added CE1, CE2, CE3: 150uF, rcl:CPOL-USE2-5
- added CON_P: LITE_TRAP_2POS, con-molex:LITE_TRAP_2POS
- added CREF: 4.7uF, Condensatori:0474_TAJA475M016RNJ
- added CRES1A: 1.2nF, rcl:C-USROUND
- added CRES1B: 1nF, rcl:C-US
- added CRES2A, CRES2B: 100pF, rcl:C-US
- added CVA, CVB: 50pF, rcl:C-TRIMM3018_11
- added ICSP10: PINHEAD-2x5-P1.27, Connettori:0171_PH127-205DF055G00AROUND-PADS
- added JPA, JPB, JP_PWR: NA, pinhead:PINHD-1X2
- added L1: 2.2uH, rcl:L-US4X4
- added R3: 10K, rcl:R-US_ROUND
- added R4, RP_INT, RP_SCL, RP_SDA: 10k, rcl:R-US_ROUND
- added RAA: 22, rcl:C-USC0805
- added RAB: 22, rcl:R-US_R0805
- added RFA, RFB: EM4095, em-microelectronic:EM4095
- added SW1: MFS201N-9-Z, switch:MFS201N-9-Z
- added VREG: LM3671, Texas Instruments:LM3671_SWITCHING_REGSOT23
- C1, C3: device Condensatori:0015_100NF_0603 -> rcl:C-USROUND
- C5: value 4.7uF -> 100nF; device Condensatori:0474_TAJA475M016RNJ -> rcl:C-USROUND
- C8: device Condensatori:0142_10NF_0603 -> rcl:C-USROUND
- ICSP6: value 3x2 M -> 3x2M
- L6, L7: device Protezione:0001_BLM21PG300SN1D_/_MH2029-300Y -> inductors:BLM15H0805
- R1: value 10k -> 100; device Resistenze:0028_CR0603JW103L -> rcl:R-US_ROUND
- R2: device Resistenze:0049_330R_0603 -> rcl:R-US_ROUND
- RTC: value RTC_PCF8523T -> MC-RTC-RV-1805-C3-I2C; device microbuilder:RTC_PCF8523T -> Microcrystal-RTC:MC-RTC-RV-1805-C3-I2C
- VDIV1: device Resistenze:2339_ -> rcl:R-US_ROUND
- VDIV2: device Resistenze:2022_CR0603FW104L -> rcl:R-US_ROUND
- Z5, Z6: value CG0603MLC-05E -> ESD_SUPRESSOR; device Protezione:0010_BRNCG0603MLC-05E -> diode:ESD_SUPRESSOR
- renumbered AD to HDR_AD, D2 to D1, HEADER_IOH to HDR_IOH, HEADER_IOL to HDR_IOL, HEADER_POWER to HDR_POWER, IC2 to MCU, ICSP to ICSP6, U$4 to SD
Connections:
- removed net +5V: HDR_POWER.5, ICSP6.2
- removed net HEADER_AD: HDR_AD.1
- removed net N$21: CNB.2, RF_B.INPUT
- removed net N$23: D4B.C, R5B.1, RF_B.COIL1
- removed net N$24: CAB.2, D1B.A, RF_B.COIL2
- removed net N$25: CAB.1, D5B.A, J3-2.S, R1B.1, R2B.2
- removed net N$26: R4B.2, RF_B.RF
- removed net N$27: C22_4.+, R3B.1, RF_B.CFE, RF_B.MS, RF_B.VS
- removed net N$28: D1B.C, D2B.C, R1B.2
- removed net N$29: D3B.A, D4B.A, R2B.1
- removed net N$30: C1B.2, D2B.A, D3B.C, R3B.2, R4B.1
- removed net N$40: CAA.2, D1A.A, RF_A.COIL2
- removed net N$41: CAA.1, D5A.A, J2-1.S, R1A.1, R2A.2
- removed net N$43: R4A.2, RF_A.RF
- removed net N$44: C22_3.+, R3A.1, RF_A.CFE, RF_A.MS, RF_A.VS
- removed net N$56: HDR_POWER.1
- new net CVB: CDIV1B.1, CRES1B.2, CRES2B.2, CVB.E, JPB.1
- new net N$16: CXB.1, RAB.2, RFB.ANT1
- new net N$6: CDC2.1, RFA.DC2
- new net N$7: CRES1B.1, CRES2B.1, CVB.A, RFB.ANT2
- new net N$8: CDIV1B.2, CDIV2B.1, RFB.DMOD_IN
- new net N$9: CDCB.1, RFB.DC2
- new net SW: L1.1, VREG.SW
- net +3V3: now also C2.2, C3.3V.1, C5.1, ICSP10.1, L1.2, R4.2, RP_INT.2, RP_SCL.2, RP_SDA.2, VREG.FB; no longer C20.1, C3.2, C3V.1, ICSP!.1, LDO.VO, R1.2, R12.2, R13.2, R9.2
- net 12_IN: now also CON_PG$2.S, JP_PWR.2; no longer U$6G$2.S
- net GND: now also BAT.-, C10.1, C11.2, C2.1, C3.2, C3.3V.2, C5.2, C5V.2, C6.2, C7.2, C9.1, CAGNDA.2, CAGNDB.2, CBLKA.2, CBLKB.2, CDC2.2, CDCB.2, CDIV2A.2, CDIV2B.2, CE1.-, CE2.-, CE3.-, CFCAPA.2, CFCAPB.2, CON_PG$1.S, CREF.-, ICSP10.3, ICSP10.5, ICSP10.9, JP_PWR.1, R3.2, RFA.DVSS, RFA.MOD, RFA.VSS, RFB.DVSS, RFB.MOD, RFB.VSS, RTC.GND, RTC.PSW, RTC.WDI, VREG.GND, Z5.P$1, Z6.P$1; no longer C12V.2, C19.2, C1A.1, C1B.1, C20.2, C21.2, C22_1.-, C22_2.-, C22_3.-, C22_4.-, C23.1, C24.1, C26.2, C2A.1, C2B.1, C3.1, C3A.1, C3B.1, C3V.2, C4.2, C5.-, G1.-, ICSP!.3, ICSP!.5, ICSP!.9, LDO.GND, R10.1, R6A.1, R6B.1, RF_A.DGND, RF_A.GND, RF_A.OE, RF_B.DGND, RF_B.GND, RF_B.OE, RTC.VSS, U$6G$1.S, Z5.2, Z6.2
- net N$1: now also R1.1; no longer R6.1
- net N$10: now also C6.1; no longer C21.1
- net N$11: now also CDECB.2, RFB.CDEC_OUT; no longer CNA.2, RF_A.INPUT
- net N$12: now also CRES1A.1, CRES2A.1, CVA.A, RFA.ANT2; no longer C2A.2, CNA.1, D5A.C, R6A.2
- net N$13: now also CDIV1A.2, CDIV2A.1, RFA.DMOD_IN; no longer C1A.2, D2A.A, D3A.C, R3A.2, R4A.1
- net N$14: now also CDIV1A.1, CRES1A.2, CRES2A.2, CVA.E, JPA.1; no longer J2-2.S, R5A.2
- net N$15: now also CDECB.1, RFB.CDEC_IN; no longer J3-1.S, R5B.2
- net N$17: now also SW1.O; no longer U$9.O
- net N$18: now also CDECA.2, RFA.CDEC_OUT; no longer D1A.C, D2A.C, R1A.2
- net N$19: now also CDECA.1, RFA.CDEC_IN; no longer C3B.2, RF_B.HIPASS
- net N$2: now also CFCAPB.1, RFB.FCAP; no longer RTC.XO, Y1.2
- net N$20: now also CXA.1, RAA.2, RFA.ANT1; no longer D3A.A, D4A.A, R2A.1
- net N$22: now also JPB.2, RAB.1; no longer C2B.2, CNB.1, D5B.C, R6B.2
- net N$3: now also CAGNDB.1, RFB.AGND; no longer RTC.XI, Y1.1
- net N$35: now also JPA.2, RAA.1; no longer D4A.C, R5A.1, RF_A.COIL1
- net N$4: now also CFCAPA.1, RFA.FCAP; no longer C22_1.+, R7.2, RF_A.VBATT, RF_B.VBATT
- net N$5: now also CAGNDA.1, RFA.AGND; no longer C3A.2, RF_A.HIPASS
- net PA00_XIN32: now also C9.2; no longer C23.2
- net PA01_XOUT32: now also C10.2; no longer C24.2
- net PA02_AIN0: now also HDR_AD.1
- net PA03_AREFA: now also C3.1, CREF.+; no longer C4.1, C5.+
- net PA21_INT&SDCS: now also RP_INT.1, RTC.CLK/INT; no longer R9.1, RTC.!INT1/CLK
- net PA22_SDA: now also RP_SDA.1; no longer R13.1
- net PA23_SCL: now also RP_SCL.1; no longer R12.1
- net PA27_TX_LED: now also R1.2; no longer R6.2
- net PA28_2FETS: now also R3.1; no longer R10.2
- net PA30_SWCLK: now also ICSP10.4; no longer ICSP!.4
- net PA31_SWDIO: now also ICSP10.2; no longer ICSP!.2
- net PA6_RFID_SHD: now also RFA.SHD; no longer RF_A.STBY
- net PA7_RFID_SHD2: now also RFB.SHD; no longer RF_B.STBY
- net PB03_RFIDIN: now also RFA.DMOD_OUT, RFB.DMOD_OUT; no longer RF_A.OUTPUT, RF_B.OUTPUT
- net RESET: now also ICSP10.10, R4.1; no longer ICSP!.10, R1.1
- net TARGET_USB_N: now also Z6.P$2; no longer Z6.1
- net TARGET_USB_P: now also Z5.P$2; no longer Z5.1
- net VBAT1: now also BAT.+, RTC.V_BAK; no longer G1.+, RTC.VBAT
- net VDDCORE: now also C11.1; no longer C19.1
- net V_IN: now also C5V.1, CBLKA.1, CBLKB.1, CE1.+, CE2.+, CE3.+, CXA.2, CXB.2, HDR_POWER.5, ICSP6.2, RFA.DVDD, RFA.VDD, RFB.DVDD, RFB.VDD, SW1.P, VREG.EN, VREG.VIN; no longer C12V.1, C22_2.+, LDO.VIN, R7.1, RF_A.DVS, RF_A.VEXT, RF_B.DVS, RF_B.VEXT, U$9.P
- net XUSB: now also C7.1, SW1.S; no longer C26.1, U$9.S
Other:
- note removed: "10"
- note removed: "11"
- note removed: "12"
- note removed: "13"
- note removed: "14"
- note removed: "15"
- note removed: "16"
- note removed: "2"
- note removed: "3"
- note removed: "4"
- note removed: "5"
- note removed: "6"
- note removed: "8"
- note removed: "9"
- note removed: "BAT"
- note removed: "CFE"
- note removed: "DGND"
- note removed: "DVS"
- note removed: "GND"
- note removed: "HIPASS"
- note removed: "INPUT"
- note removed: "MS"
- note removed: "OE"
- note removed: "OUTPUT"
- note removed: "RF"
- note removed: "STBY"
- note removed: "VEXT"
- note removed: "VS"
